File: DNA_macropad.kicad_sch (KiCad schematic)
At the start: 21 parts

Commit message: Finished electrical schematic
Parts:
- removed R? (x2): 22 Ω, symbol Device:R_Small_US
- added D1, D2, D3, D4: SOD-123, Diode_SMD:D_SOD-123, symbol Device:D_Small
- added J1: AVR-ISP-6, random-keyboard-parts:Reset_Pretty-Mask, symbol Connector:AVR-ISP-6
- added MX1: A, MX_Alps_Hybrid:MX-1U, symbol MX_Alps_Hybrid:MX-NoLED
- added MX2: C, MX_Alps_Hybrid:MX-1U, symbol MX_Alps_Hybrid:MX-NoLED
- added MX3: T/U, MX_Alps_Hybrid:MX-1U, symbol MX_Alps_Hybrid:MX-NoLED
- added MX4: G, MX_Alps_Hybrid:MX-1U, symbol MX_Alps_Hybrid:MX-NoLED
- C1, C2, C3, C4, C5, C6, C7: renamed from C?; footprint (none) -> Capacitor_SMD:C_0805_2012Metric
- F1: renamed from F?; footprint (none) -> Fuse:Fuse_1206_3216Metric
- R1, R2, R3, R4, R7, R8: renamed from R?; footprint (none) -> Resistor_SMD:R_0805_2012Metric
- SW1: renamed from SW?; footprint (none) -> random-keyboard-parts:SKQG-1155865
- U1: renamed from U?; footprint (none) -> random-keyboard-parts:SOT143B
- USB1: renamed from USB?; footprint (none) -> Type-C:HRO-TYPE-C-31-M-12
- Y1: renamed from Y?; footprint (none) -> Crystal:Crystal_SMD_3225-4Pin_3.2x2.5mm
- gave numbers to parts that had none: 1
Connections:
- net +5V: now also J1.2 (VCC)
- net D+: now also U2.4 (D+)
- net D-: now also U2.3 (D-)
- net GND: now also J1.6 (GND)
- net RESET: now reaches R7.2, SW1.2, U2.13 (~{RESET})
- net RESET: now also J1.5 (~{RST})
- net MISO: now reaches U2.10 (PB2)
- net MISO: now also J1.1 (MISO)
- net MISI: now reaches U2.11 (PB3)
- net MISI: now also J1.4 (MOSI)
- net ROW0: now reaches U2.27 (PD7)
- net ROW0: now also D1.1 (K), D3.1 (K)
- net COL1: now reaches U2.28 (PB4)
- net COL1: now also MX3.1 (COL), MX4.1 (COL)
- net COL0: now reaches U2.29 (PB5)
- net COL0: now also MX1.1 (COL), MX2.1 (COL)
- net ROW1: now reaches U2.30 (PB6)
- net ROW1: now also D2.1 (K), D4.1 (K)
- net SCK: now reaches U2.9 (PB1)
- net SCK: now also J1.3 (SCK)
- new net: D4.2 (A), MX4.2 (ROW)
- new net: D1.2 (A), MX1.2 (ROW)
- new net: D2.2 (A), MX2.2 (ROW)
- new net: D3.2 (A), MX3.2 (ROW)
- no-connect marks 3 -> 21
Other:
- moved on the sheet: C4, C5, C6, C7, R3, R7, SW1
